Commit message: [miniquad] tmp debugging

File: resources/robots/miniquad/miniquad.urdf (robot description, URDF)
Before this commit: robot multirotor, 9 links, 8 joints
Links:
- link arm_motor_0: geometry visual cylinder length=0.1202081528 radius=0.01
- link arm_motor_1: geometry visual cylinder length=0.1202081528 radius=0.01
- link arm_motor_2: geometry visual cylinder length=0.1202081528 radius=0.01
- link arm_motor_3: geometry visual cylinder length=0.1202081528 radius=0.01
- link base_link: mass 0.321 -> 0.860
Joints:
- joint base_link_to_arm_motor_0: origin xyz=0.08 -0.08 0.0 rpy=-1.5707963267948968 2.220446049250313e-16 -2.3561944901923453 -> xyz=0.0425 -0.0425 0.0 rpy=-1.5707963267948968 2.220446049250313e-16 -2.3561944901923453
- joint base_link_to_arm_motor_1: origin xyz=-0.08 -0.08 0.0 rpy=1.5707963267948968 2.220446049250313e-16 -0.7853981633974482 -> xyz=-0.0425 -0.0425 0.0 rpy=1.5707963267948968 2.220446049250313e-16 -0.7853981633974482
- joint base_link_to_arm_motor_2: origin xyz=-0.08 0.08 0.0 rpy=1.5707963267948968 0.0 -2.3561944901923453 -> xyz=-0.0425 0.0425 0.0 rpy=1.5707963267948968 0.0 -2.3561944901923453
- joint base_link_to_arm_motor_3: origin xyz=0.08 0.08 0.0 rpy=-1.5707963267948968 0.0 -0.7853981633974482 -> xyz=0.0425 0.0425 0.0 rpy=-1.5707963267948968 0.0 -0.7853981633974482
- joint base_link_to_motor_0: origin xyz=0.16 -0.16 0.0 rpy=0.0 0.0 0.0 -> xyz=0.085 -0.085 0.026 rpy=0.0 0.0 0.0
- joint base_link_to_motor_1: origin xyz=-0.16 -0.16 0.0 rpy=0.0 0.0 0.0 -> xyz=-0.085 -0.085 0.026 rpy=0.0 0.0 0.0
- joint base_link_to_motor_2: origin xyz=-0.16 0.16 0.0 rpy=0.0 0.0 0.0 -> xyz=-0.085 0.085 0.026 rpy=0.0 0.0 0.0
- joint base_link_to_motor_3: origin xyz=0.16 0.16 0.0 rpy=0.0 0.0 0.0 -> xyz=0.085 0.085 0.026 rpy=0.0 0.0 0.0
